File: pcb/volumer_v0.2/rp2040.kicad_sch (KiCad schematic)
At the start: 27 parts, among them SW1 TS-3025-B-C-B, SW2 TS-3025-B-C-B, U3 W25Q128JVS, U4 RP2040, U8 LD1117S33TR, Y2 12Mhz

Commit message: Added finished v0.2 PCB
Parts:
- C14, C31, C32, C33, C34, C35, C38, C39, C40, C41, C42, C43: footprint Capacitor_SMD:C_0201_0603Metric -> Capacitor_SMD:C_0603_1608Metric
- C18: footprint Capacitor_SMD:C_0402_1005Metric -> Capacitor_SMD:C_0603_1608Metric; LCSC C15525 -> C19702
- C36, C37: footprint Capacitor_SMD:C_0402_1005Metric -> Capacitor_SMD:C_0603_1608Metric; LCSC C52923 -> C15849
- R29, R31: footprint Resistor_SMD:R_0402_1005Metric -> Resistor_SMD:R_0603_1608Metric; LCSC C25744 -> C25804
- R30, R34: footprint Resistor_SMD:R_0402_1005Metric -> Resistor_SMD:R_0603_1608Metric; LCSC C11702 -> C21190
- R32, R33: value 27 -> 33; footprint Resistor_SMD:R_0402_1005Metric -> Resistor_SMD:R_0603_1608Metric; LCSC (none) -> C23140
Changed lines of the file:
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@@
       (effects (font (size 1.27 1.27)) (justify left))
     )
-    (property "Footprint" "Capacitor_SMD:C_0201_0603Metric" (at 226.06 39.37 0)
+    (property "Footprint" "Capacitor_SMD:C_0603_1608Metric" (at 226.06 39.37 0)
       (effects (font (size 1.27 1.27)) hide)
     )
@@
       (effects (font (size 1.27 1.27)))
     )
-    (property "Footprint" "Resistor_SMD:R_0402_1005Metric" (at 87.63 109.22 0)
+    (property "Footprint" "Resistor_SMD:R_0603_1608Metric" (at 87.63 109.22 0)
       (effects (font (size 1.27 1.27)) hide)
     )
@@
       (effects (font (size 1.27 1.27)) hide)
     )
-    (property "LCSC" "C11702" (at 87.63 109.22 0)
+    (property "LCSC" "C21190" (at 87.63 109.22 0)
       (effects (font (size 1.27 1.27)) hide)
     )
@@
       (effects (font (size 1.27 1.27)))
     )
-    (property "Value" "27" (at 161.29 61.595 90)
-      (effects (font (size 1.27 1.27)))
-    )
-    (property "Footprint" "Resistor_SMD:R_0402_1005Metric" (at 163.83 63.5 0)
+    (property "Value" "33" (at 161.29 61.595 90)
+      (effects (font (size 1.27 1.27)))
+    )
+    (property "Footprint" "Resistor_SMD:R_0603_1608Metric" (at 163.83 63.5 0)
       (effects (font (size 1.27 1.27)) hide)
     )
@@
       (effects (font (size 1.27 1.27)) hide)
     )
+    (property "LCSC" "C23140" (at 163.83 63.5 0)
+      (effects (font (size 1.27 1.27)) hide)
+    )
     (pin "1")
     (pin "2")
@@
       (effects (font (size 1.27 1.27)))
     )
-    (property "Value" "27" (at 161.29 67.945 90)
-      (effects (font (size 1.27 1.27)))
-    )
-    (property "Footprint" "Resistor_SMD:R_0402_1005Metric" (at 163.83 66.04 0)
+    (property "Value" "33" (at 161.29 67.945 90)
+      (effects (font (size 1.27 1.27)))
+    )
+    (property "Footprint" "Resistor_SMD:R_0603_1608Metric" (at 163.83 66.04 0)
       (effects (font (size 1.27 1.27)) hide)
     )
@@
       (effects (font (size 1.27 1.27)) hide)
     )
+    (property "LCSC" "C23140" (at 163.83 66.04 0)
+      (effects (font (size 1.27 1.27)) hide)
+    )
     (pin "1")
     (pin "2")
@@
       (effects (font (size 1.27 1.27)) (justify left))
     )
-    (property "Footprint" "Capacitor_SMD:C_0402_1005Metric" (at 219.71 39.37 0)
+    (property "Footprint" "Capacitor_SMD:C_0603_1608Metric" (at 219.71 39.37 0)
       (effects (font (size 1.27 1.27)) hide)
     )
@@
       (effects (font (size 1.27 1.27)) hide)
     )
-    (property "LCSC" "C52923" (at 219.71 39.37 0)
+    (property "LCSC" "C15849" (at 219.71 39.37 0)
       (effects (font (size 1.27 1.27)) hide)
     )
@@
       (effects (font (size 1.27 1.27)) (justify left))
     )
-    (property "Footprint" "Capacitor_SMD:C_0201_0603Metric" (at 257.81 39.37 0)
+    (property "Footprint" "Capacitor_SMD:C_0603_1608Metric" (at 257.81 39.37 0)
       (effects (font (size 1.27 1.27)) hide)
     )
@@
       (effects (font (size 1.27 1.27)))
     )
-    (property "Footprint" "Resistor_SMD:R_0402_1005Metric" (at 153.67 111.76 0)
+    (property "Footprint" "Resistor_SMD:R_0603_1608Metric" (at 153.67 111.76 0)
       (effects (font (size 1.27 1.27)) hide)
     )
@@
       (effects (font (size 1.27 1.27)) hide)
     )
-    (property "LCSC" "C11702" (at 153.67 111.76 0)
+    (property "LCSC" "C21190" (at 153.67 111.76 0)
       (effects (font (size 1.27 1.27)) hide)
     )
@@
       (effects (font (size 1.27 1.27)) (justify left))
     )
-    (property "Footprint" "Capacitor_SMD:C_0402_1005Metric" (at 189.23 39.37 0)
+    (property "Footprint" "Capacitor_SMD:C_0603_1608Metric" (at 189.23 39.37 0)
       (effects (font (size 1.27 1.27)) hide)
     )
@@
       (effects (font (size 1.27 1.27)) hide)
     )
-    (property "LCSC" "C52923" (at 189.23 39.37 0)
+    (property "LCSC" "C15849" (at 189.23 39.37 0)
       (effects (font (size 1.27 1.27)) hide)
     )
@@
       (effects (font (size 1.27 1.27)) (justify left))
     )
-    (property "Footprint" "Capacitor_SMD:C_0201_0603Metric" (at 245.11 39.37 0)
+    (property "Footprint" "Capacitor_SMD:C_0603_1608Metric" (at 245.11 39.37 0)
       (effects (font (size 1.27 1.27)) hide)
     )
@@
       (effects (font (size 1.27 1.27)) (justify left))
     )
-    (property "Footprint" "Capacitor_SMD:C_0201_0603Metric" (at 232.41 39.37 0)
+    (property "Footprint" "Capacitor_SMD:C_0603_1608Metric" (at 232.41 39.37 0)
       (effects (font (size 1.27 1.27)) hide)
     )
@@
       (effects (font (size 1.27 1.27)) (justify left))
     )
-    (property "Footprint" "Resistor_SMD:R_0402_1005Metric" (at 135.89 50.8 0)
+    (property "Footprint" "Resistor_SMD:R_0603_1608Metric" (at 135.89 50.8 0)
       (effects (font (size 1.27 1.27)) hide)
     )
@@
       (effects (font (size 1.27 1.27)) hide)
     )
-    (property "LCSC" "C25744" (at 135.89 50.8 0)
+    (property "LCSC" "C25804" (at 135.89 50.8 0)
       (effects (font (size 1.27 1.27)) hide)
     )
@@
       (effects (font (size 1.27 1.27)) (justify left))
     )
-    (property "Footprint" "Capacitor_SMD:C_0402_1005Metric" (at 73.66 52.07 0)
+    (property "Footprint" "Capacitor_SMD:C_0603_1608Metric" (at 73.66 52.07 0)
       (effects (font (size 1.27 1.27)) hide)
     )
@@
       (effects (font (size 1.27 1.27)) hide)
     )
-    (property "LCSC" "C15525" (at 73.66 52.07 0)
+    (property "LCSC" "C19702" (at 73.66 52.07 0)
       (effects (font (size 1.27 1.27)) hide)
     )
@@
       (effects (font (size 1.27 1.27)))
     )
-    (property "Footprint" "Resistor_SMD:R_0402_1005Metric" (at 67.31 97.79 0)
+    (property "Footprint" "Resistor_SMD:R_0603_1608Metric" (at 67.31 97.79 0)
       (effects (font (size 1.27 1.27)) hide)
     )
@@
       (effects (font (size 1.27 1.27)) hide)
     )
-    (property "LCSC" "C25744" (at 67.31 97.79 0)
+    (property "LCSC" "C25804" (at 67.31 97.79 0)
       (effects (font (size 1.27 1.27)) hide)
     )
@@
       (effects (font (size 1.27 1.27)) (justify left))
     )
-    (property "Footprint" "Capacitor_SMD:C_0201_0603Metric" (at 182.88 39.37 0)
+    (property "Footprint" "Capacitor_SMD:C_0603_1608Metric" (at 182.88 39.37 0)
       (effects (font (size 1.27 1.27)) hide)
     )
@@
       (effects (font (size 1.27 1.27)) (justify left))
     )
-    (property "Footprint" "Capacitor_SMD:C_0201_0603Metric" (at 238.76 39.37 0)
+    (property "Footprint" "Capacitor_SMD:C_0603_1608Metric" (at 238.76 39.37 0)
       (effects (font (size 1.27 1.27)) hide)
     )
@@
       (effects (font (size 1.27 1.27)) (justify left))
     )
-    (property "Footprint" "Capacitor_SMD:C_0201_0603Metric" (at 129.54 118.11 0)
+    (property "Footprint" "Capacitor_SMD:C_0603_1608Metric" (at 129.54 118.11 0)
       (effects (font (size 1.27 1.27)) hide)
     )
@@
       (effects (font (size 1.27 1.27)) (justify left))
     )
-    (property "Footprint" "Capacitor_SMD:C_0201_0603Metric" (at 139.7 118.11 0)
+    (property "Footprint" "Capacitor_SMD:C_0603_1608Metric" (at 139.7 118.11 0)
       (effects (font (size 1.27 1.27)) hide)
     )
@@
       (effects (font (size 1.27 1.27)) (justify left))
     )
-    (property "Footprint" "Capacitor_SMD:C_0201_0603Metric" (at 251.46 39.37 0)
+    (property "Footprint" "Capacitor_SMD:C_0603_1608Metric" (at 251.46 39.37 0)
       (effects (font (size 1.27 1.27)) hide)
     )
@@
       (effects (font (size 1.27 1.27)) (justify left))
     )
-    (property "Footprint" "Capacitor_SMD:C_0201_0603Metric" (at 38.1 111.76 0)
+    (property "Footprint" "Capacitor_SMD:C_0603_1608Metric" (at 38.1 111.76 0)
       (effects (font (size 1.27 1.27)) hide)
     )
@@
       (effects (font (size 1.27 1.27)) (justify left))
     )
-    (property "Footprint" "Capacitor_SMD:C_0201_0603Metric" (at 53.34 52.07 0)
+    (property "Footprint" "Capacitor_SMD:C_0603_1608Metric" (at 53.34 52.07 0)
       (effects (font (size 1.27 1.27)) hide)
     )
@@
       (effects (font (size 1.27 1.27)) (justify left))
     )
-    (property "Footprint" "Capacitor_SMD:C_0201_0603Metric" (at 176.53 39.37 0)
-      (effects (font (size 1.27 1.27)) hide)
-    )
+    (property "Footprint" "Capacitor_SMD:C_0603_1608Metric" (at 176.53 39.37 0)
+      (effects (font (size 1.27 1.27)) hide)
+    )
