File: pcb/volumer_v0.2/volumer_v02.kicad_pcb (KiCad board)
At the start: 4 copper layers, 90 x 80 mm, 39 parts, among them SW1 TS-3025-B-C-B, SW2 TS-3025-B-C-B, U1 W25Q128JVS, U2 LD1117S33TR, U3 RP2040, Y1 12Mhz

Commit message: Added finished v0.2 PCB
Parts:
- C1, C10, C11, C12, C13, C14, C15, C2, C4, C5, C6, C7: footprint Capacitor_SMD:C_0201_0603Metric -> Capacitor_SMD:C_0603_1608Metric
- C3, C8, C9: footprint Capacitor_SMD:C_0402_1005Metric -> Capacitor_SMD:C_0603_1608Metric
- R1, R2, R3, R4, R5, R6: footprint Resistor_SMD:R_0402_1005Metric -> Resistor_SMD:R_0603_1608Metric
- R7, R8: value 27 -> 33; footprint Resistor_SMD:R_0402_1005Metric -> Resistor_SMD:R_0603_1608Metric
- moved C6 10.9 mm to (180.9, 74.4), turned to 180 degrees
- moved C11 8.76 mm to (180.9, 71.1), turned to 180 degrees
- moved C5 3.19 mm to (187.9, 82.0)
- moved C10 2.71 mm to (195.0, 67.0)
- moved C14 2.60 mm to (195.0, 68.6)
- moved C7 2.26 mm to (190.4, 78.2)
- moved Y1 2.16 mm to (184.9, 82.0)
- moved R3 1.92 mm to (175.8, 60.9)
- moved R4 1.73 mm to (177.5, 63.7)
- moved C9 1.67 mm to (192.7, 65.7)
- moved C3 1.55 mm to (194.0, 62.4)
- moved C12 1.44 mm to (180.9, 69.5)
- moved C13 1.38 mm to (180.9, 72.7)
- moved C15 1.24 mm to (187.8, 78.1)
- moved C4 1.22 mm to (183.7, 77.3)
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Routing:
- net GND: track 18.2 -> 26.8 mm, vias 27 -> 28
- net +3V3: track 29.9 -> 38.2 mm
- net /rp2040/1V1: track 18.3 -> 25.5 mm, vias 3 -> 5
- net /rp2040/XIN: track 7.66 -> 13.6 mm
- net /rp2040/QSPI_SS: track 13.7 -> 16.1 mm
- net /rp2040/~{USB_BOOT}: track 38.2 -> 36.5 mm
- net Net-(USB1-CC2): track 1.41 -> 2.46 mm
- net Net-(C5-Pad1): track 3.18 -> 4.17 mm
- net Net-(USB1-CC1): track 1.58 -> 2.48 mm
- net /USB_D+: track 16.6 -> 16.0 mm
- net /rp2040/XOUT: track 2.08 -> 2.62 mm
