File: pcb/volumer_v0.2/volumer_v02.kicad_sch (KiCad schematic)
At the start: 11 parts

Commit message: Added finished v0.2 PCB
Parts:
- R1, R2: footprint Resistor_SMD:R_0402_1005Metric -> Resistor_SMD:R_0603_1608Metric; LCSC C25905 -> C23186
Changed lines of the file:
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@@
       (effects (font (size 1.27 1.27)) (justify left))
     )
-    (property "Footprint" "Resistor_SMD:R_0402_1005Metric" (at 67.31 42.545 0)
+    (property "Footprint" "Resistor_SMD:R_0603_1608Metric" (at 67.31 42.545 0)
       (effects (font (size 1.27 1.27)) hide)
     )
@@
       (effects (font (size 1.27 1.27)) hide)
     )
-    (property "LCSC" "C25905" (at 67.31 42.545 0)
+    (property "LCSC" "C23186" (at 67.31 42.545 0)
       (effects (font (size 1.27 1.27)) hide)
     )
@@
       (effects (font (size 1.27 1.27)) (justify left))
     )
-    (property "Footprint" "Resistor_SMD:R_0402_1005Metric" (at 74.295 42.545 0)
+    (property "Footprint" "Resistor_SMD:R_0603_1608Metric" (at 74.295 42.545 0)
       (effects (font (size 1.27 1.27)) hide)
     )
@@
       (effects (font (size 1.27 1.27)) hide)
     )
-    (property "LCSC" "C25905" (at 74.295 42.545 0)
-      (effects (font (size 1.27 1.27)) hide)
-    )
+    (property "LCSC" "C23186" (at 74.295 42.545 0)
+      (effects (font (size 1.27 1.27)) hide)
+    )
